File: RFID_Reader.kicad_pcb (KiCad board)
At the start: 2 copper layers, 57.9 x 67.9 mm, 17 parts, among them J1 Conn_01x04_Female, J2 Barrel_Jack, J3 Conn_01x08_Female, SW1 SW_Push, SW2 SW_Push, SW3 SW_Push, U1 WeMos_D1_mini

Commit message: - add bom, step and schematic as PDF
Parts:
- SW1, SW2, SW3: footprint Button_Switch_THT:SW_PUSH_6mm_H8mm -> Button_Switch_THT:SW_PUSH_6mm_H9.5mm
